File: Board/SlimeVR_Dock.kicad_sch (KiCad schematic)
At the start: 31 parts, among them J1Fan1 Conn_01x04_Pin, J1Temp1 Conn_01x05_Pin, J1_Control1 Conn_01x03_Pin, J1_MainPW1 USB_C_Receptacle_USB2.0_16P, J1_Monitor1 Conn_01x03_Pin, J1_Prog1 Conn_01x03_Pin, Q1 NDT452AP, Q6 BC817, U1 ESP32-C3-WROOM-02, U17 74HC165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

Commit message: Version 3
Hopefully it works idk ?:D
Connections:
- net Earth: now also U17.10 (DS)
- no-connect marks 12 -> 11
Changed lines of the file:
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@@
 	(title_block
 		(title "SlimeVR Dock")
-		(date "2026-04-10")
-		(rev "1.0")
+		(date "2026-05-16")
+		(rev "2.0")
 		(company "Skaut0071")
 	)
@@
 	)
 	(no_connect
-		(at 146.05 26.67)
-	)
-	(no_connect
 		(at 50.8 144.78)
 	)
@@
 	(wire
 		(pts
+			(xy 144.78 21.59) (xy 140.97 21.59)
+		)
+		(stroke
+			(width 0)
+			(type default)
+		)
+	)
+	(wire
+		(pts
 			(xy 53.34 109.22) (xy 53.34 114.3)
 		)
@@
 	(wire
 		(pts
+			(xy 144.78 26.67) (xy 144.78 21.59)
+		)
+		(stroke
+			(width 0)
+			(type default)
+		)
+	)
+	(wire
+		(pts
 			(xy 55.88 144.78) (xy 55.88 128.27)
 		)
@@
 	(wire
 		(pts
+			(xy 140.97 21.59) (xy 140.97 22.86)
+		)
+		(stroke
+			(width 0)
+			(type default)
+		)
+	)
+	(wire
+		(pts
 			(xy 50.8 114.3) (xy 53.34 114.3)
 		)
@@
 		)
 	)
+	(wire
+		(pts
+			(xy 146.05 26.67) (xy 144.78 26.67)
+		)
+		(stroke
+			(width 0)
+			(type default)
+		)
+	)
 	(bus
 		(pts
@@
 					(unit 1)
 				)
+			)
+		)
+	)
+	(symbol
+		(lib_id "power:Earth")
+		(at 140.97 22.86 0)
+		(unit 1)
+		(body_style 1)
+		(exclude_from_sim no)
+		(in_bom yes)
+		(on_board yes)
+		(in_pos_files yes)
+		(dnp no)
+		(property "Reference" "#PWR0117"
+			(at 140.97 29.21 0)
+			(hide yes)
+			(show_name no)
+			(do_not_autoplace no)
+			(effects
+				(font
+					(size 1.27 1.27)
+				)
+			)
+		)
+		(property "Value" "Earth"
+			(at 140.97 26.924 0)
+			(show_name no)
+			(do_not_autoplace no)
+			(effects
+				(font
+					(size 1.27 1.27)
+				)
+			)
+		)
+		(property "Footprint" ""
+			(at 140.97 22.86 0)
+			(hide yes)
+			(show_name no)
+			(do_not_autoplace no)
+			(effects
+				(font
+					(size 1.27 1.27)
+				)
+			)
+		)
+		(property "Datasheet" ""
+			(at 140.97 22.86 0)
+			(hide yes)
+			(show_name no)
+			(do_not_autoplace no)
+			(effects
+				(font
+					(size 1.27 1.27)
+				)
+			)
+		)
+		(property "Description" "Power symbol creates a global label with name \"Earth\""
+			(at 140.97 22.86 0)
+			(hide yes)
+			(show_name no)
+			(do_not_autoplace no)
+			(effects
+				(font
+					(size 1.27 1.27)
+				)
+			)
+		)
+		(pin "1"
+		)
+		(instances
+			(project "SlimeVR_Dock"
+				(path "/06ff9557-1f9b-4670-8a34-bb7684a016dd"
+					(reference "#PWR0117")
+					(unit 1)
+				)
