File: Board/SlimeVR_Dock.kicad_sch (KiCad schematic)
At the start: 31 parts, among them J1Fan1 Conn_01x04_Pin, J1Temp1 Conn_01x05_Pin, J1_Control1 Conn_01x03_Pin, J1_MainPW1 USB_C_Receptacle_USB2.0_16P, J1_Monitor1 Conn_01x03_Pin, J1_Prog1 Conn_01x03_Pin, Q1 NDT452AP, Q6 BC817, U1 ESP32-C3-WROOM-02, U17 74HC165, U18 74HC165, U19 74HC595, U2 CH224K, U3 XC6220B331MR

Commit message: Fixing from Review
Parts:
- added D2: 10V, symbol Device:D_Zener
- added R59: 10k, Resistor_SMD:R_0603_1608Metric, symbol Device:R
- added R60: 1k, Resistor_SMD:R_0603_1608Metric, symbol Device:R
Connections:
- net +3V3: now also U19.10 (~{SRCLR}), R59.2
- net +5V: no longer U19.10 (~{SRCLR})
- net Boot: now also U19.13 (~{OE})
- net Earth: now also D2.2 (A); no longer U19.13 (~{OE})
- net GET: now also R59.1
- net at Q1.1 (G), R3.1: now also D2.1 (K), R60.2; no longer U2.10 (PG)
- new net: R60.1, U2.10 (PG)

Commit message: V4 review update
- new review from from this version alreaady done
Parts:
- D2: footprint (none) -> Diode_SMD:D_0603_1608Metric
Changed lines of the file:
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@@
 			)
 		)
-		(property "Footprint" ""
+		(property "Footprint" "Diode_SMD:D_0603_1608Metric"
 			(at 72.39 106.68 0)
 			(hide yes)

Commit message: Small updates from review
- Updated Revisions
Parts:
- R1: footprint Resistor_SMD:R_0603_1608Metric -> Resistor_SMD:R_2010_5025Metric
Connections:
- net at U18.10 (DS): now also U17.9 (Q7); no longer U17.7 (~{Q7})
Changed lines of the file:
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@@
 		(title "SlimeVR Dock")
 		(date "2026-05-16")
-		(rev "2.0")
+		(rev "3.0")
 		(company "Skaut0071")
 	)
@@
 	)
 	(no_connect
-		(at 171.45 26.67)
+		(at 201.93 31.75)
 	)
 	(no_connect
-		(at 201.93 31.75)
+		(at 171.45 29.21)
 	)
 	(no_connect
@@
 	(wire
 		(pts
-			(xy 171.45 29.21) (xy 176.53 29.21)
-		)
-		(stroke
-			(width 0)
-			(type default)
-		)
-	)
-	(wire
-		(pts
 			(xy 77.47 44.45) (xy 77.47 69.85)
 		)
@@
 	(wire
 		(pts
+			(xy 171.45 26.67) (xy 173.99 26.67)
+		)
+		(stroke
+			(width 0)
+			(type default)
+		)
+	)
+	(wire
+		(pts
 			(xy 163.83 142.24) (xy 163.83 143.51)
 		)
@@
 	(wire
 		(pts
+			(xy 173.99 29.21) (xy 176.53 29.21)
+		)
+		(stroke
+			(width 0)
+			(type default)
+		)
+	)
+	(wire
+		(pts
 			(xy 232.41 64.77) (xy 232.41 60.96)
 		)
@@
 	(wire
 		(pts
+			(xy 173.99 26.67) (xy 173.99 29.21)
+		)
+		(stroke
+			(width 0)
+			(type default)
+		)
+	)
+	(wire
+		(pts
 			(xy 271.78 123.19) (xy 271.78 125.73)
 		)
@@
 			)
 		)
-		(property "Footprint" "Resistor_SMD:R_0603_1608Metric"
+		(property "Footprint" "Resistor_SMD:R_2010_5025Metric"
 			(at 59.69 114.808 90)
 			(hide yes)

Commit message: New review completed version
-Board ONLY changes no documentation updated YET
Parts:
- removed J1Temp1: Conn_01x05_Pin, Connector_PinHeader_2.54mm:PinHeader_1x04_P2.54mm_Vertical, symbol Connector:Conn_01x05_Pin
- added C43, C44, C45, C46, C47: 100nF, Capacitor_SMD:C_0603_1608Metric, symbol Device:C
- added J1Temp1: Conn_01x04_Pin, Connector_PinHeader_2.54mm:PinHeader_1x04_P2.54mm_Vertical, symbol Connector:Conn_01x04_Pin
- added R61, R62: 10k, Resistor_SMD:R_0603_1608Metric, symbol Device:R
Connections:
- net +3V3: now also C43.1, C44.2, C45.2, C46.1, J1Temp1.1 (Pin_1), R61.1, R62.2
- net Earth: now also C43.2, C44.1, C45.1, C46.2, C47.2, J1Temp1.2 (Pin_2)
- net Enable: now also C47.1
- net SCL: now also J1Temp1.3 (Pin_3)
- net SDA: now also J1Temp1.4 (Pin_4)
- net at U1.16 (IO2): now also R62.1
- net at U1.7 (IO8): now also R61.2
- no-connect marks 11 -> 8
Other:
- note added: "I use BME280 module"
- note removed: "I use TC74A0 in TO-220 footprint"
- moved on the sheet: C10, C11, C12, C13, J1_Control1, J1_Monitor1, J1_Prog1, R17, R18, R23, R24, R59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

Commit message: Some traces angle changes and all LCSC codes added
Parts:
- BZ1: LCSC (none) -> alr
- C1: LCSC (none) -> alr C15849
- C10, C12: LCSC (none) -> alr C19702
- C11, C13: LCSC (none) -> alr C100040
- C43, C44, C45, C46, C47: LCSC (none) -> alr C6119867
- D1, D2: LCSC (none) -> pls find idk
- J1Fan1, J1Temp1, J1_Control1, J1_Monitor1, J1_Prog1: LCSC (none) -> x
- J1_MainPW1: LCSC C5178539 -> alr C5178539
- Q1: LCSC C274614 -> alr C274614
- Q6: LCSC C39828 -> alr C39828
- R1: LCSC (none) -> C2974087
- R17, R18, R2, R3, R4, R42, R59, R61, R62: LCSC (none) -> alr C98220
- R23, R24: LCSC (none) -> alr C99782
- R33, R60: LCSC (none) -> alr C22548
- U17, U18: LCSC C5613 -> alr C5613
- U19: LCSC C5947 -> alr C5947
- U2: LCSC C970725 -> alr C970725
- U3: LCSC C86534 -> alr C86534

Commit message: updated diod footprint
Parts:
- D1: footprint Diode_SMD:D_0603_1608Metric -> Diode_SMD:D_SOD-323; LCSC pls find idk -> alr C7473299
- D2: footprint Diode_SMD:D_0603_1608Metric -> Diode_SMD:D_SOD-123; LCSC pls find idk -> alr C47117498
Changed lines of the file:
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@@
 			)
 		)
-		(property "Footprint" "Diode_SMD:D_0603_1608Metric"
+		(property "Footprint" "Diode_SMD:D_SOD-123"
 			(at 72.39 106.68 0)
 			(hide yes)
@@
 			)
 		)
-		(property "LCSC" "pls find idk"
+		(property "LCSC" "alr C47117498"
 			(at 72.39 106.68 0)
 			(hide yes)
@@
 			)
 		)
-		(property "Footprint" "Diode_SMD:D_0603_1608Metric"
+		(property "Footprint" "Diode_SMD:D_SOD-323"
 			(at 229.87 88.9 0)
 			(hide yes)
@@
 			)
 		)
-		(property "LCSC" "pls find idk"
+		(property "LCSC" "alr C7473299"
 			(at 229.87 88.9 0)
 			(hide yes)

Commit message: Updated bom
Parts:
- BZ1: LCSC alr -> alr - Any passive buzzer
- J1Fan1: LCSC x -> alr C240840
- J1Temp1, J1_Control1, J1_Monitor1, J1_Prog1: LCSC x -> x - Only holes
Changed lines of the file:
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@@
 			)
 		)
-		(property "LCSC" "x"
+		(property "LCSC" "x - Only holes"
 			(at 236.22 26.67 90)
 			(hide yes)
@@
 			)
 		)
-		(property "LCSC" "x"
+		(property "LCSC" "x - Only holes"
 			(at 195.58 85.09 0)
 			(hide yes)
@@
 			)
 		)
-		(property "LCSC" "alr"
+		(property "LCSC" "alr - Any passive buzzer"
 			(at 229.87 85.09 90)
 			(hide yes)
@@
 			)
 		)
-		(property "LCSC" "x"
+		(property "LCSC" "x - Only holes"
 			(at 195.58 99.06 0)
 			(hide yes)
@@
 			)
 		)
-		(property "LCSC" "x"
+		(property "LCSC" "alr C240840"
 			(at 234.95 55.88 90)
 			(hide yes)
@@
 			)
 		)
-		(property "LCSC" "x"
+		(property "LCSC" "x - Only holes"
 			(at 200.66 115.57 0)
 			(hide yes)
