File: Board/USB-C.kicad_sch (KiCad schematic)
At the start: 2 parts, among them J2 USB_C_Receptacle_USB2.0_16P, U6 INA226

Commit message: Conecting usb to esp
added in/out and out/in reistry
Changed lines of the file:
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@@
 	(wire
 		(pts
-			(xy 128.27 91.44) (xy 128.27 97.79)
+			(xy 128.27 95.25) (xy 128.27 97.79)
 		)
 		(stroke
@@
 	(wire
 		(pts
-			(xy 129.54 91.44) (xy 128.27 91.44)
+			(xy 129.54 95.25) (xy 128.27 95.25)
 		)
 		(stroke
@@
 	(hierarchical_label "CC_Line"
 		(shape bidirectional)
-		(at 129.54 91.44 0)
+		(at 129.54 95.25 0)
 		(effects
 			(font

Commit message: Finished Schematic
Parts:
- added C14: 10uF, Capacitor_SMD:C_0603_1608Metric, symbol Device:C
- added R25: 10m, Resistor_SMD:R_0603_1608Metric, symbol Device:R
- J2: footprint (none) -> Library:CONN_USB4145-03-0230-C_GCT
Connections:
- net +3V3: now also C14.1
- net Earth: now also J2.A1 (GND), J2.A12 (GND), J2.B1 (GND), J2.B12 (GND), J2.S1 (SHIELD), C14.2
- net VBUS: now also U6.10 (Vin+), R25.1
- net A1: now reaches U6.1 (A1)
- net at J2.A4 (VBUS), J2.A9 (VBUS), J2.B4 (VBUS)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: now also U6.9 (Vin-), R25.2; no longer U6.10 (Vin+)
- net A0: now reaches U6.2 (A0)
Other:
- note added: "Conector and OverCharge"
- moved on the sheet: J2, U6

Commit message: Updavení USB-C
Other:
- note added: "Conector and Current Mesure"
- note removed: "Conector and OverCharge"
Changed lines of the file:
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@@
 	(generator_version "9.0")
 	(paper "A4")
-	(text "Conector and OverCharge "
+	(text "Conector and Current Mesure"
 		(exclude_from_sim no)
-		(at 155.702 132.08 0)
+		(at 152.146 132.334 0)
 		(effects
 			(font

Commit message: Complete
-fixed tach pullup missing
- may have some unrecognised issues
Parts:
- J2: footprint Library:CONN_USB4145-03-0230-C_GCT -> Library:YTC-TC16S-128
Changed lines of the file:
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@@
 			)
 		)
-		(property "Footprint" "Library:CONN_USB4145-03-0230-C_GCT"
+		(property "Footprint" "Library:YTC-TC16S-128"
 			(at 127 99.06 0)
 			(effects

Commit message: Updated fields for LCSC
Parts:
- J2: LCSC (none) -> C2927282
- U6: LCSC (none) -> C49851
Changed lines of the file:
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@@
+			)
+		)
+		(property "LCSC" "C49851"
+			(at 170.18 105.41 0)
+			(effects
+				(font
+					(size 1.27 1.27)
+				)
+				(hide yes)
 			)
 		)
@@
 			(at 123.19 99.06 0)
 			(effects
+				(font
+					(size 1.27 1.27)
+				)
+				(hide yes)
+			)
+		)
+		(property "LCSC" "C2927282"
+			(at 123.19 99.06 0)
+			(effects

Commit message: Version 3
Hopefully it works idk ?:D
Parts:
- C14: value 10uF -> 100nF
Changed lines of the file:
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@@
+	(wire
+		(pts
+			(xy 181.61 113.03) (xy 180.34 113.03)
+		)
+		(stroke
+			(width 0)
+			(type default)
+		)
+	)
 	(wire
 		(pts
@@
 	(hierarchical_label "ALERT"
 		(shape output)
-		(at 180.34 113.03 0)
+		(at 181.61 113.03 0)
 		(effects
 			(font
@@
 			)
 		)
-		(property "Value" "10uF"
+		(property "Value" "100nF"
 			(at 160.02 87.6299 0)
 			(show_name no)
