File: Board/USB-C.kicad_sch (KiCad schematic)
At the start: 5 parts, among them J2 USB_C_Receptacle_USB2.0_16P, U6 INA226

Commit message: Fixing from Review
Parts:
- R25: value 10m -> 50m
Changed lines of the file:
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@@
 			)
 		)
-		(property "Value" "10m"
+		(property "Value" "50m"
 			(at 155.956 109.22 0)
 			(show_name no)

Commit message: Board and schema update
curent mesuring resistors swap for bigger
some more grounding was done
Parts:
- R25: footprint Resistor_SMD:R_0603_1608Metric -> Resistor_SMD:R_0805_2012Metric
Changed lines of the file:
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@@
 			)
 		)
-		(property "Footprint" "Resistor_SMD:R_0603_1608Metric"
+		(property "Footprint" "Resistor_SMD:R_0805_2012Metric"
 			(at 153.162 107.95 90)
 			(hide yes)

Commit message: New review completed version
-Board ONLY changes no documentation updated YET
Other:
- company: (none) -> Skaut0071
- title: (none) -> Overcurent proteciton
Changed lines of the file:
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@@
 	(generator_version "10.0")
 	(paper "A4")
+	(title_block
+		(title "Overcurent proteciton")
+		(date "2026-09-21")
+		(rev "1.2")
+		(company "Skaut0071")
+	)
 	(text "Conector and Current Mesure"
 		(exclude_from_sim no)

Commit message: Some traces angle changes and all LCSC codes added
Parts:
- C14, C28: LCSC (none) -> alr C6119867
- R25: LCSC (none) -> C42389461
- U6: LCSC C49851 -> alr C49851
Changed lines of the file:
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@@
 			)
 		)
-		(property "LCSC" "C49851"
+		(property "LCSC" "alr C49851"
 			(at 170.18 105.41 0)
 			(hide yes)
@@
 			)
 		)
+		(property "LCSC" "alr C6119867"
+			(at 149.86 116.84 0)
+			(hide yes)
+			(show_name no)
+			(do_not_autoplace no)
+			(effects
+				(font
+					(size 1.27 1.27)
+				)
+			)
+		)
 		(pin "1"
 		)
@@
 		)
 		(property "Description" "Resistor"
+			(at 154.94 107.95 0)
+			(hide yes)
+			(show_name no)
+			(do_not_autoplace no)
+			(effects
+				(font
+					(size 1.27 1.27)
+				)
+			)
+		)
+		(property "LCSC" "C42389461"
 			(at 154.94 107.95 0)
 			(hide yes)
@@
 			(at 163.83 86.36 0)
 			(hide yes)
+			(show_name no)
+			(do_not_autoplace no)
+			(effects
+				(font
+					(size 1.27 1.27)
+				)
+			)
+		)
+		(property "LCSC" "alr C6119867"
+			(at 163.83 86.36 0)
+			(hide yes)

Commit message: updated diod footprint
Parts:
- J2: LCSC C2927282 -> alr C2927282
Changed lines of the file:
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@@
 			)
 		)
-		(property "LCSC" "C2927282"
+		(property "LCSC" "alr C2927282"
 			(at 123.19 99.06 0)
 			(hide yes)
