File: Board/DUSBSS.kicad_sch (KiCad schematic)
At the start: 11 parts, among them Q2 BC857, U5 AP22652W6-7

Commit message: Fixing from Review
Parts:
- removed R50: 10k, Resistor_SMD:R_0603_1608Metric, symbol Device:R
- added R51: 10k, symbol Device:R
Connections:
- net +3V3: now also R51.2
- net EN: now also R51.1

Commit message: V4 review update
- new review from from this version alreaady done
Parts:
- R51: footprint (none) -> Resistor_SMD:R_0603_1608Metric
Changed lines of the file:
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@@
 			)
 		)
-		(property "Footprint" ""
+		(property "Footprint" "Resistor_SMD:R_0603_1608Metric"
 			(at 177.8 65.278 90)
 			(hide yes)

Commit message: more checking and added detailed review
Parts:
- R6: value 10k -> 18k
Changed lines of the file:
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@@
 			)
 		)
-		(property "Value" "10k"
+		(property "Value" "18k"
 			(at 119.126 70.866 90)
 			(show_name no)

Commit message: Small updates from review
- Updated Revisions
Parts:
- R6: value 18k -> 14.3k
Changed lines of the file:
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@@
 			)
 		)
-		(property "Value" "18k"
-			(at 119.126 70.866 90)
+		(property "Value" "14.3k"
+			(at 118.11 70.866 90)
 			(show_name no)
 			(do_not_autoplace no)

Commit message: New review completed version
-Board ONLY changes no documentation updated YET
Other:
- company: (none) -> Skaut0071
- title: (none) -> Dual USB-C charger monitoring
Changed lines of the file:
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@@
 	(generator_version "10.0")
 	(paper "A4")
+	(title_block
+		(title "Dual USB-C charger monitoring")
+		(date "2026-09-21")
+		(rev "1.8")
+		(company "Skaut0071")
+	)
 	(text "Protection and Detection"
 		(exclude_from_sim no)

Commit message: Some traces angle changes and all LCSC codes added
Parts:
- C2, C3: LCSC (none) -> alr C19702
- Q2: LCSC C111644 -> alr C111644
- R19, R38, R46, R5, R51, R7: LCSC (none) -> alr C98220
- R6: LCSC (none) -> ?alr? C3017492
- U5: LCSC C2158038 -> alr C2158038
Changed lines of the file:
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@@
+			)
+		)
+		(property "LCSC" "alr C98220"
+			(at 177.8 63.5 90)
+			(hide yes)
+			(show_name no)
+			(do_not_autoplace no)
+			(effects
+				(font
+					(size 1.27 1.27)
+				)
 			)
 		)
@@
 			)
 		)
+		(property "LCSC" "?alr? C3017492"
+			(at 120.65 68.58 90)
+			(hide yes)
+			(show_name no)
+			(do_not_autoplace no)
+			(effects
+				(font
+					(size 1.27 1.27)
+				)
+			)
+		)
 		(pin "2"
 		)
@@
 		)
 		(property "Description" "Resistor"
+			(at 143.51 100.33 0)
+			(hide yes)
+			(show_name no)
+			(do_not_autoplace no)
+			(effects
+				(font
+					(size 1.27 1.27)
+				)
+			)
+		)
+		(property "LCSC" "alr C98220"
 			(at 143.51 100.33 0)
 			(hide yes)
@@
 			)
 		)
+		(property "LCSC" "alr C19702"
+			(at 181.61 74.93 0)
+			(hide yes)
+			(show_name no)
+			(do_not_autoplace no)
+			(effects
+				(font
+					(size 1.27 1.27)
+				)
+			)
+		)
 		(pin "2"
 		)
@@
 			)
 		)
+		(property "LCSC" "alr C98220"
+			(at 125.73 110.49 0)
+			(hide yes)
+			(show_name no)
+			(do_not_autoplace no)
+			(effects
+				(font
+					(size 1.27 1.27)
+				)
+			)
+		)
 		(pin "1"
 		)
@@
 			)
 		)
+		(property "LCSC" "alr C19702"
+			(at 128.27 80.01 0)
+			(hide yes)
+			(show_name no)
+			(do_not_autoplace no)
+			(effects
+				(font
+					(size 1.27 1.27)
+				)
+			)
+		)
 		(pin "2"
 		)
@@
 			)
 		)
+		(property "LCSC" "alr C98220"
+			(at 138.43 120.65 0)
+			(hide yes)
+			(show_name no)
+			(do_not_autoplace no)
+			(effects
+				(font
+					(size 1.27 1.27)
+				)
+			)
+		)
 		(pin "1"
 		)
@@
 			)
 		)
-		(property "LCSC" "C111644"
+		(property "LCSC" "alr C111644"
 			(at 132.08 118.11 90)
 			(hide yes)
@@
 			)
 		)
+		(property "LCSC" "alr C98220"
+			(at 140.97 137.16 0)
+			(hide yes)
+			(show_name no)
+			(do_not_autoplace no)
+			(effects
+				(font
+					(size 1.27 1.27)
+				)
+			)
+		)
 		(pin "1"
 		)
@@
 			)
 		)
+		(property "LCSC" "alr C98220"
+			(at 120.65 60.96 90)
+			(hide yes)
+			(show_name no)
+			(do_not_autoplace no)
+			(effects
+				(font
+					(size 1.27 1.27)
+				)
+			)
+		)
 		(pin "1"
 		)
@@
 			)
 		)
-		(property "LCSC" "C2158038"
+		(property "LCSC" "alr C2158038"
 			(at 170.18 71.12 0)
 			(hide yes)

Commit message: found correct LCSC code for 14.3k
Parts:
- R6: LCSC ?alr? C3017492 -> C22799
Changed lines of the file:
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@@
 			)
 		)
-		(property "LCSC" "?alr? C3017492"
+		(property "LCSC" "C22799"
 			(at 120.65 68.58 90)
 			(hide yes)
