File: Board/DUSBSS.kicad_sch (KiCad schematic)
At the start: 11 parts, among them Q2 BC857, U5 AP22652W6-7

Commit message: Final check
Parts:
- R6: value 14.3k -> 13k; LCSC C22799 -> C54920854
Changed lines of the file:
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@@
 			)
 		)
-		(property "Value" "14.3k"
-			(at 118.11 70.866 90)
+		(property "Value" "13k"
+			(at 118.618 70.866 90)
 			(show_name no)
 			(do_not_autoplace no)
@@
 			)
 		)
-		(property "LCSC" "C22799"
+		(property "LCSC" "C54920854"
 			(at 120.65 68.58 90)
 			(hide yes)
