File: Board/StepDown.kicad_sch (KiCad schematic)
At the start: 26 parts, among them U4 TPS548A20RVER

Commit message: Updates LCSC codes
Parts:
- C40: footprint Capacitor_SMD:C_1210_3225Metric -> Capacitor_SMD:C_0603_1608Metric
Changed lines of the file:
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@@
 			)
 		)
-		(property "Footprint" "Capacitor_SMD:C_1210_3225Metric"
+		(property "Footprint" "Capacitor_SMD:C_0603_1608Metric"
 			(at 116.84 93.0148 0)
 			(hide yes)

Commit message: Some traces angle changes and all LCSC codes added
Parts:
- C22, C23, C24, C25, C26, C30, C31: LCSC (none) -> alr C16780
- C27: LCSC (none) -> C1743
- C29: LCSC (none) -> alr C98192
- C39: LCSC (none) -> alr C49678
- C40: LCSC (none) -> alr C15849
- C41: value 0.1uF -> 0.1nF; LCSC (none) -> alr C49678
- C42: LCSC (none) -> C1531
- L1: LCSC (none) -> C49261221
- R34, R37, R41: LCSC (none) -> alr C2907067
- R35, R57: LCSC (none) -> alr C98220
- R36: LCSC (none) -> C2907011
- R39: LCSC (none) -> alr C2907038
- R40: LCSC (none) -> alr C4197
- R54: LCSC (none) -> C17660
- R55: LCSC (none) -> C2907006
- R56: LCSC (none) -> alr C14675
- U4: LCSC (none) -> alr C90084

Commit message: Final check
Parts:
- C22, C23, C30: LCSC alr C16780 -> alr C47117451
- C40: LCSC alr C15849 -> C15849
- C41: value 0.1nF -> 100nF
- L1: footprint Inductor_SMD:L_Coilcraft_XAL7070-XXX -> Library:L_Coilank_APS0730
- R39: value 43k -> 36k; LCSC alr C2907038 -> C54531400
- U4: LCSC alr C90084 -> alr C468255
Changed lines of the file:
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@@
 			)
 		)
-		(property "Footprint" "Inductor_SMD:L_Coilcraft_XAL7070-XXX"
+		(property "Footprint" "Library:L_Coilank_APS0730"
 			(at 179.07 93.98 0)
 			(hide yes)
@@
 			)
 		)
-		(property "LCSC" "alr C90084"
+		(property "LCSC" "alr C468255"
 			(at 146.05 109.22 0)
 			(hide yes)
@@
 			)
 		)
-		(property "Value" "43k"
+		(property "Value" "36k"
 			(at 115.062 108.712 90)
 			(show_name no)
@@
 			)
 		)
-		(property "LCSC" "alr C2907038"
+		(property "LCSC" "C54531400"
 			(at 116.84 106.68 90)
 			(hide yes)
@@
 			)
 		)
-		(property "LCSC" "alr C15849"
+		(property "LCSC" "C15849"
 			(at 113.03 93.98 90)
 			(hide yes)
@@
 			)
 		)
-		(property "Value" "0.1nF"
+		(property "Value" "100nF"
 			(at 171.45 81.534 0)
 			(show_name no)
@@
 			)
 		)
-		(property "LCSC" "alr C16780"
+		(property "LCSC" "alr C47117451"
 			(at 118.11 73.66 90)
 			(hide yes)
@@
 			)
 		)
-		(property "LCSC" "alr C16780"
+		(property "LCSC" "alr C47117451"
 			(at 118.11 64.77 90)
 			(hide yes)
@@
 			)
 		)
-		(property "LCSC" "alr C16780"
+		(property "LCSC" "alr C47117451"
 			(at 118.11 82.55 90)
 			(hide yes)

Commit message: removed unused files
Parts:
- C40: LCSC C15849 -> alr C15849
Changed lines of the file:
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@@
 			)
 		)
-		(property "LCSC" "C15849"
+		(property "LCSC" "alr C15849"
 			(at 113.03 93.98 90)
 			(hide yes)
